File: pcb/Audio_True_Bypass_Stereo.kicad_sch (KiCad schematic)
At the start: 12 parts, among them J2 AUDIO_IN_TRS, J4 AUDIO_OUT_TRS, K1 G6K-2, K2 G6K-2, Q1 SS8050, U5 CPC1018N, U6 CPC1018N

Commit message: Updated kiCad FIles
Parts:
- J2, J4: footprint NMJ6HCD2:NEUTRIK_NMJ6HCD2 -> Connector_Audio:Jack_6.35mm_Neutrik_NMJ6HCD2_Horizontal
Connections:
- net GND: no longer J2.R, J2.RN, J2.SN, J2.T, J2.TN, J4.R, J4.RN, J4.SN, J4.T, J4.TN, K1.4, K1.6, K1.7, K2.4, K2.6, K2.7, U5.4, U6.4
- new net AUDIO_IN_JACK_LEFT: J2.T, K1.4, K1.7
- new net AUDIO_IN_JACK_RIGHT: J2.R, K2.4, K2.7
- new net AUDIO_OUT_JACK_LEFT: J4.T, K1.6, U5.4
- new net AUDIO_OUT_JACK_RIGHT: J4.R, K2.6, U6.4
Other:
- moved on the sheet: J2, J4

Commit message: Lots of updates to Schematic and pcb design
Parts:
- J2, J4: footprint Connector_Audio:Jack_6.35mm_Neutrik_NMJ6HCD2_Horizontal -> NMJ6HCD2:NEUTRIK_NMJ6HCD2
Connections:
- net +5V renamed +5VA
Changed lines of the file:
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@@
-	)
-	(symbol
-		(lib_id "power:+5V")
-		(at 135.89 40.64 0)
-		(unit 1)
-		(exclude_from_sim no)
-		(in_bom yes)
-		(on_board yes)
-		(dnp no)
-		(fields_autoplaced yes)
-		(property "Reference" "#PWR041"
-			(at 135.89 44.45 0)
-			(effects
-				(font
-					(size 1.27 1.27)
-				)
-				(hide yes)
-			)
-		)
-		(property "Value" "+5V"
-			(at 135.89 35.56 0)
-			(effects
-				(font
-					(size 1.27 1.27)
-				)
-			)
-		)
-		(property "Footprint" ""
-			(at 135.89 40.64 0)
-			(effects
-				(font
-					(size 1.27 1.27)
-				)
-				(hide yes)
-			)
-		)
-		(property "Datasheet" ""
-			(at 135.89 40.64 0)
-			(effects
-				(font
-					(size 1.27 1.27)
-				)
-				(hide yes)
-			)
-		)
-		(property "Description" ""
-			(at 135.89 40.64 0)
-			(effects
-				(font
-					(size 1.27 1.27)
-				)
-			)
-		)
-		(pin "1"
-		)
-		(instances
-			(project "DaisySeedPedal125b"
-				(path "/1d54e6f4-7c7a-4f03-b2db-a136bdff5b99/d5b1af0e-2179-4bcd-8e24-55fd6680ab7e"
-					(reference "#PWR041")
-					(unit 1)
-				)
-			)
-		)
 	)
 	(symbol
@@
 			)
 		)
-		(property "Footprint" "Connector_Audio:Jack_6.35mm_Neutrik_NMJ6HCD2_Horizontal"
+		(property "Footprint" "NMJ6HCD2:NEUTRIK_NMJ6HCD2"
 			(at 220.98 76.2 0)
 			(effects
@@
 	)
 	(symbol
+		(lib_id "power:+5VA")
+		(at 135.89 40.64 0)
+		(unit 1)
+		(exclude_from_sim no)
+		(in_bom yes)
+		(on_board yes)
+		(dnp no)
+		(fields_autoplaced yes)
+		(property "Reference" "#PWR050"
+			(at 135.89 44.45 0)
+			(effects
+				(font
+					(size 1.27 1.27)
+				)
+				(hide yes)
+			)
+		)
+		(property "Value" "+5VA"
+			(at 135.89 35.56 0)
+			(effects
+				(font
+					(size 1.27 1.27)
+				)
+			)
+		)
+		(property "Footprint" ""
+			(at 135.89 40.64 0)
+			(effects
+				(font
+					(size 1.27 1.27)
+				)
+				(hide yes)
+			)
+		)
+		(property "Datasheet" ""
+			(at 135.89 40.64 0)
+			(effects
+				(font
+					(size 1.27 1.27)
+				)
+				(hide yes)
+			)
+		)
+		(property "Description" "Power symbol creates a global label with name \"+5VA\""
+			(at 135.89 40.64 0)
+			(effects
+				(font
+					(size 1.27 1.27)
+				)
+				(hide yes)
+			)
+		)
+		(pin "1"
+		)
+		(instances
+			(project ""
+				(path "/1d54e6f4-7c7a-4f03-b2db-a136bdff5b99/d5b1af0e-2179-4bcd-8e24-55fd6680ab7e"
+					(reference "#PWR050")
+					(unit 1)
+				)
+			)
+		)
+	)
+	(symbol
 		(lib_id "power:GND")
 		(at 82.55 190.5 0)
@@
 			)
 		)
-		(property "Footprint" "Connector_Audio:Jack_6.35mm_Neutrik_NMJ6HCD2_Horizontal"
+		(property "Footprint" "NMJ6HCD2:NEUTRIK_NMJ6HCD2"
 			(at 240.03 124.46 0)
 			(effects

Commit message: Updates
Connections:
- net GND: now also J2.RN, J2.SN, J2.TN, J4.RN, J4.SN, J4.TN
Changed lines of the file:
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@@
+	)
+	(junction
+		(at 231.14 132.08)
+		(diameter 0)
+		(color 0 0 0 0)
 	)
 	(junction
@@
 	)
 	(junction
+		(at 231.14 83.82)
+		(diameter 0)
+		(color 0 0 0 0)
+	)
+	(junction
 		(at 135.89 104.14)
 		(diameter 0)
@@
 	)
 	(junction
+		(at 231.14 129.54)
+		(diameter 0)
+		(color 0 0 0 0)
+	)
+	(junction
+		(at 231.14 124.46)
+		(diameter 0)
+		(color 0 0 0 0)
+	)
+	(junction
+		(at 231.14 76.2)
+		(diameter 0)
+		(color 0 0 0 0)
+	)
+	(junction
 		(at 135.89 46.99)
 		(diameter 0)
@@
 		(color 0 0 0 0)
 	)
+	(junction
+		(at 231.14 81.28)
+		(diameter 0)
+		(color 0 0 0 0)
+	)
 	(wire
 		(pts
@@
 	(wire
 		(pts
+			(xy 228.6 71.12) (xy 231.14 71.12)
+		)
+		(stroke
+			(width 0)
+			(type default)
+		)
+	)
+	(wire
+		(pts
 			(xy 227.33 132.08) (xy 227.33 134.62)
 		)
@@
 	(wire
 		(pts
+			(xy 228.6 81.28) (xy 231.14 81.28)
+		)
+		(stroke
+			(width 0)
+			(type default)
+		)
+	)
+	(wire
+		(pts
 			(xy 106.68 185.42) (xy 106.68 140.97)
 		)
@@
 	(wire
 		(pts
+			(xy 231.14 124.46) (xy 231.14 129.54)
+		)
+		(stroke
+			(width 0)
+			(type default)
+		)
+	)
+	(wire
+		(pts
 			(xy 111.76 104.14) (xy 111.76 120.65)
 		)
@@
 	(wire
 		(pts
+			(xy 228.6 76.2) (xy 231.14 76.2)
+		)
+		(stroke
+			(width 0)
+			(type default)
+		)
+	)
+	(wire
+		(pts
 			(xy 104.14 83.82) (xy 116.84 83.82)
 		)
@@
 	(wire
 		(pts
+			(xy 231.14 71.12) (xy 231.14 76.2)
+		)
+		(stroke
+			(width 0)
+			(type default)
+		)
+	)
+	(wire
+		(pts
 			(xy 228.6 127) (xy 232.41 127)
 		)
@@
 	(wire
 		(pts
+			(xy 231.14 119.38) (xy 231.14 124.46)
+		)
+		(stroke
+			(width 0)
+			(type default)
+		)
+	)
+	(wire
+		(pts
 			(xy 120.65 46.99) (xy 111.76 46.99)
 		)
@@
 	(wire
 		(pts
+			(xy 231.14 76.2) (xy 231.14 81.28)
+		)
+		(stroke
+			(width 0)
+			(type default)
+		)
+	)
+	(wire
+		(pts
 			(xy 132.08 120.65) (xy 135.89 120.65)
 		)
@@
 	(wire
 		(pts
+			(xy 231.14 132.08) (xy 232.41 132.08)
+		)
+		(stroke
+			(width 0)
+			(type default)
+		)
+	)
+	(wire
+		(pts
 			(xy 111.76 63.5) (xy 111.76 95.25)
 		)
@@
 	(wire
 		(pts
-			(xy 227.33 132.08) (xy 232.41 132.08)
+			(xy 227.33 132.08) (xy 231.14 132.08)
 		)
 		(stroke
@@
 	(wire
 		(pts
+			(xy 231.14 81.28) (xy 231.14 83.82)
+		)
+		(stroke
+			(width 0)
+			(type default)
+		)
+	)
+	(wire
+		(pts
 			(xy 132.08 143.51) (xy 151.13 143.51)
 		)
@@
 	(wire
 		(pts
-			(xy 228.6 83.82) (xy 233.68 83.82)
+			(xy 228.6 83.82) (xy 231.14 83.82)
 		)
 		(stroke
@@
 	(wire
 		(pts
+			(xy 231.14 129.54) (xy 231.14 132.08)
+		)
+		(stroke
+			(width 0)
+			(type default)
+		)
+	)
+	(wire
+		(pts
 			(xy 134.62 76.2) (xy 134.62 78.74)
 		)
@@
 	(wire
 		(pts
+			(xy 231.14 129.54) (xy 232.41 129.54)
+		)
+		(stroke
+			(width 0)
+			(type default)
+		)
+	)
+	(wire
+		(pts
 			(xy 132.08 63.5) (xy 135.89 63.5)
 		)
@@
 	(wire
 		(pts
+			(xy 231.14 124.46) (xy 232.41 124.46)
+		)
+		(stroke
+			(width 0)
+			(type default)
+		)
+	)
+	(wire
+		(pts
 			(xy 135.89 46.99) (xy 135.89 63.5)
 		)
@@
 		)
 		(stroke
+			(width 0)
+			(type default)
+		)
+	)
+	(wire
+		(pts
+			(xy 231.14 83.82) (xy 233.68 83.82)
+		)
+		(stroke
+			(width 0)
+			(type default)
+		)
+	)
+	(wire
+		(pts
+			(xy 232.41 119.38) (xy 231.14 119.38)
+		)
+		(stroke
